File: Hardware/LedDriver4x.kicad_pcb (KiCad board)
At the start: 2 copper layers, 44.4 x 34.9 mm, 14 parts, among them J1 Barrel_Jack, J2 Conn_01x03, U1 TPS92511

Commit message: Post Review Changes
Changes per request of John Fritz
Parts:
- added J3: Conn_01x02, Pin_Headers:Pin_Header_Angled_1x02_Pitch2.54mm, F.Cu at (175.9, 77.5)
- added J4: Conn_01x02, Pin_Headers:Pin_Header_Angled_1x02_Pitch2.54mm, F.Cu at (175.9, 83.8)
- J2: value Conn_01x03 -> Conn_01x02; footprint Pin_Headers:Pin_Header_Angled_1x03_Pitch2.54mm -> Pin_Headers:Pin_Header_Angled_1x02_Pitch2.54mm
- moved C2 9.92 mm to (173.4, 78.7)
- moved J2 6.49 mm to (175.9, 71.1)
- moved L1 5.25 mm to (166.4, 79.4), turned to 270 degrees
- moved D1 4.58 mm to (157.5, 77.5), turned to 0 degrees
Connections:
- J2 pad 1: LEDCATH -> +48V
- J2 pad 2: LEDANODE -> GND
Routing:
- net +48V: track 13.0 -> 26.6 mm
- net LEDANODE: track 21.9 -> 10.1 mm
- net Net-(FB1-Pad2): track 7.76 -> 10.6 mm
- net Net-(D1-Pad2): track 5.14 -> 3.85 mm
- net DIM: track 21.2 -> 22.2 mm
- net LEDCATH: track 60.3 -> 60.8 mm
Other:
- board text added: "Nathan Snyder 48V in 36V out LED Driver 300mA Current Limit 12/4/2017 Rev 1.0"

Commit message: Stuff
things
Parts:
- L1: footprint Inductors_THT:L_Axial_L20.0mm_D8.0mm_P5.08mm_Vertical -> Inductors_THT:L_Radial_D8.7mm_P5.00mm_Fastron_07HCP
- moved C1 3.05 mm to (146.1, 83.8)
- moved R2 1.27 mm to (158.8, 87.6)
- moved R1 1.02 mm to (148.6, 86.2)
Routing:
- net Net-(C1-Pad1): track 7.98 -> 4.96 mm
- net Net-(R2-Pad1): track 3.72 -> 2.45 mm
- net Net-(R1-Pad1): track 3.40 -> 2.38 mm
