File: Hardware/LedDriver4x.sch (KiCad schematic (older format))
At the start: 14 parts, among them J1 Barrel_Jack, J2 Conn_01x03, U1 TPS92511

Commit message: Post Review Changes
Changes per request of John Fritz
Parts:
- removed J2: Conn_01x03, Pin_Headers:Pin_Header_Angled_1x03_Pitch2.54mm, symbol Conn_01x03
- added J2, J3, J4: Conn_01x02, Pin_Headers:Pin_Header_Angled_1x02_Pitch2.54mm, symbol Conn_01x02
Connections:
- net +48V: now also J2.1 (Pin_1)
- net DIM: now also J4.1 (Pin_1)
- net GND: now also J2.2 (Pin_2), J4.2 (Pin_2)
- net LEDANODE: now also J3.2 (Pin_2)
- net LEDCATH: now also J3.1 (Pin_1)
Changed lines of the file:
@@
 	1    0    0    -1
 $EndComp
-Wire Wire Line
-	4100 4200 4000 4200
-Wire Wire Line
-	4000 4200 4000 4400
-Wire Wire Line
-	4100 4050 3900 4050
-Wire Wire Line
-	4100 3750 3700 3750
-Wire Wire Line
-	3700 3950 3700 4400
-Wire Wire Line
-	4100 3900 3800 3900
-Wire Wire Line
-	3800 3900 3800 4400
-Wire Wire Line
-	3900 4250 3900 4400
-Wire Wire Line
-	5100 4200 5200 4200
-Wire Wire Line
-	5200 4400 5200 4450
-Wire Wire Line
-	5100 3900 5400 3900
-Wire Wire Line
-	5600 3900 5650 3900
-Wire Wire Line
-	5650 3650 5650 4100
-Wire Wire Line
-	5650 3100 5650 3450
-Wire Wire Line
-	5200 3300 7150 3300
-Wire Wire Line
-	5300 3500 5300 3600
-Wire Wire Line
-	5300 3800 5300 3900
-Connection ~ 5300 3900
-Wire Wire Line
-	5200 3300 5200 3750
-Wire Wire Line
-	5200 3750 5100 3750
-Connection ~ 5300 3300
-Wire Wire Line
-	7500 3450 7500 3300
-Wire Wire Line
-	7350 3300 7850 3300
-Wire Wire Line
-	6250 3300 6250 3450
-Connection ~ 6900 3300
-Connection ~ 5650 3300
-Connection ~ 6250 3300
-Wire Wire Line
-	6250 3650 6250 3850
-Wire Wire Line
-	6900 3650 6900 3850
-Wire Wire Line
-	7500 3650 7500 3850
-Wire Wire Line
-	7850 3300 7850 3200
-Connection ~ 7500 3300
-Wire Wire Line
-	5100 4050 5200 4050
-Wire Wire Line
-	5800 3100 5650 3100
-Wire Wire Line
-	5650 4100 5800 4100
-Connection ~ 5650 3900
 $Comp
 L +48V #PWR010
@@
 	1    0    0    -1
 $EndComp
-Text GLabel 9600 3800 0    60   Input ~ 0
+Text GLabel 9650 4150 0    60   Input ~ 0
 DIM
-Wire Wire Line
-	6900 3300 6900 3450
-$Comp
-L Conn_01x03 J2
-U 1 1 59D4BA5D
-P 9900 3650
-F 0 "J2" H 9900 3950 50  0000 C CNN
-F 1 "Conn_01x03" H 9900 3350 50  0000 C CNN
-F 2 "Pin_Headers:Pin_Header_Angled_1x03_Pitch2.54mm" H 9900 3650 50  0001 C CNN
-F 3 "" H 9900 3650 50  0001 C CNN
-	1    9900 3650
-	1    0    0    -1
-$EndComp
-Text GLabel 9600 3500 0    60   Input ~ 0
+Text GLabel 9600 3750 0    60   Input ~ 0
 LEDCATH
-Text GLabel 9600 3650 0    60   Input ~ 0
+Text GLabel 9600 3900 0    60   Input ~ 0
 LEDANODE
 $Comp
@@
 	1    0    0    -1
 $EndComp
-Wire Wire Line
-	9700 3550 9700 3500
-Wire Wire Line
-	9700 3500 9600 3500
-Wire Wire Line
-	9700 3650 9600 3650
-Wire Wire Line
-	9700 3750 9700 3800
-Wire Wire Line
-	9700 3800 9600 3800
 $Comp
 L Barrel_Jack J1
@@
 	-1   0    0    -1
 $EndComp
+$Comp
+L Conn_01x02 J4
+U 1 1 5A25024E
+P 9900 4150
+F 0 "J4" H 9900 4250 50  0000 C CNN
+F 1 "Conn_01x02" H 9900 3950 50  0000 C CNN
+F 2 "Pin_Headers:Pin_Header_Angled_1x02_Pitch2.54mm" H 9900 4150 50  0001 C CNN
+F 3 "" H 9900 4150 50  0001 C CNN
+	1    9900 4150
+	1    0    0    -1
+$EndComp
+$Comp
+L GND #PWR012
+U 1 1 5A2502B3
+P 9650 4300
+F 0 "#PWR012" H 9650 4050 50  0001 C CNN
+F 1 "GND" H 9650 4150 50  0000 C CNN
+F 2 "" H 9650 4300 50  0001 C CNN
+F 3 "" H 9650 4300 50  0001 C CNN
+	1    9650 4300
+	1    0    0    -1
+$EndComp
+$Comp
+L GND #PWR013
+U 1 1 5A2502EB
+P 9650 3500
+F 0 "#PWR013" H 9650 3250 50  0001 C CNN
+F 1 "GND" H 9650 3350 50  0000 C CNN
+F 2 "" H 9650 3500 50  0001 C CNN
+F 3 "" H 9650 3500 50  0001 C CNN
+	1    9650 3500
+	1    0    0    -1
+$EndComp
+$Comp
+L Conn_01x02 J3
+U 1 1 5A25043A
+P 9900 3750
+F 0 "J3" H 9900 3850 50  0000 C CNN
+F 1 "Conn_01x02" H 9900 3550 50  0000 C CNN
+F 2 "Pin_Headers:Pin_Header_Angled_1x02_Pitch2.54mm" H 9900 3750 50  0001 C CNN
+F 3 "" H 9900 3750 50  0001 C CNN
+	1    9900 3750
+	1    0    0    -1
+$EndComp
+$Comp
+L Conn_01x02 J2
+U 1 1 5A2504A3
+P 9900 3350
+F 0 "J2" H 9900 3450 50  0000 C CNN
+F 1 "Conn_01x02" H 9900 3150 50  0000 C CNN
+F 2 "Pin_Headers:Pin_Header_Angled_1x02_Pitch2.54mm" H 9900 3350 50  0001 C CNN
+F 3 "" H 9900 3350 50  0001 C CNN
+	1    9900 3350
+	1    0    0    -1
+$EndComp
+Wire Wire Line
+	4100 4200 4000 4200
+Wire Wire Line
+	4000 4200 4000 4400
+Wire Wire Line
+	4100 4050 3900 4050
+Wire Wire Line
+	4100 3750 3700 3750
+Wire Wire Line
+	3700 3950 3700 4400
+Wire Wire Line
+	4100 3900 3800 3900
+Wire Wire Line
+	3800 3900 3800 4400
+Wire Wire Line
+	3900 4250 3900 4400
+Wire Wire Line
+	5100 4200 5200 4200
+Wire Wire Line
+	5200 4400 5200 4450
+Wire Wire Line
+	5100 3900 5400 3900
+Wire Wire Line
+	5600 3900 5650 3900
+Wire Wire Line
+	5650 3650 5650 4100
+Wire Wire Line
+	5650 3100 5650 3450
+Wire Wire Line
+	5200 3300 7150 3300
+Wire Wire Line
+	5300 3500 5300 3600
+Wire Wire Line
+	5300 3800 5300 3900
+Connection ~ 5300 3900
+Wire Wire Line
+	5200 3300 5200 3750
+Wire Wire Line
+	5200 3750 5100 3750
+Connection ~ 5300 3300
+Wire Wire Line
+	7500 3450 7500 3300
+Wire Wire Line
+	7350 3300 7850 3300
+Wire Wire Line
+	6250 3300 6250 3450
+Connection ~ 6900 3300
+Connection ~ 5650 3300
+Connection ~ 6250 3300
+Wire Wire Line
+	6250 3650 6250 3850
+Wire Wire Line
+	6900 3650 6900 3850
+Wire Wire Line
+	7500 3650 7500 3850
+Wire Wire Line
+	7850 3300 7850 3200
+Connection ~ 7500 3300
+Wire Wire Line
+	5100 4050 5200 4050
+Wire Wire Line
+	5800 3100 5650 3100
+Wire Wire Line
+	5650 4100 5800 4100
+Connection ~ 5650 3900
+Wire Wire Line
+	6900 3300 6900 3450
 Wire Wire Line
 	9450 2900 9400 2900
@@
 Wire Wire Line
 	9400 2800 9400 2750
+Wire Wire Line
+	9700 4150 9650 4150
+Wire Wire Line
+	9700 4250 9650 4250
+Wire Wire Line
+	9650 4250 9650 4300
+Wire Wire Line
+	9700 3450 9650 3450
+Wire Wire Line
+	9650 3450 9650 3500
+Wire Wire Line
+	9700 3750 9600 3750
+Wire Wire Line
+	9600 3900 9650 3900
+Wire Wire Line
+	9650 3900 9650 3850
+Wire Wire Line
+	9650 3850 9700 3850
+$Comp
+L +48V #PWR014
+U 1 1 5A250A06
+P 9650 3300
+F 0 "#PWR014" H 9650 3150 50  0001 C CNN
+F 1 "+48V" H 9650 3440 50  0000 C CNN
+F 2 "" H 9650 3300 50  0001 C CNN
+F 3 "" H 9650 3300 50  0001 C CNN
+	1    9650 3300
+	1    0    0    -1
+$EndComp
+Wire Wire Line
+	9700 3350 9650 3350
+Wire Wire Line
+	9650 3350 9650 3300
 $EndSCHEMATC

Commit message: Stuff
things
Parts:
- L1: footprint Inductors_THT:L_Axial_L20.0mm_D8.0mm_P5.08mm_Vertical -> Inductors_THT:L_Radial_D8.7mm_P5.00mm_Fastron_07HCP
Changed lines of the file:
@@
 F 0 "L1" H 5530 3940 50  0000 L CNN
 F 1 "100uH" H 5530 3860 50  0000 L CNN
-F 2 "Inductors_THT:L_Axial_L20.0mm_D8.0mm_P5.08mm_Vertical" H 5500 3900 50  0001 C CNN
+F 2 "Inductors_THT:L_Radial_D8.7mm_P5.00mm_Fastron_07HCP" H 5500 3900 50  0001 C CNN
 F 3 "" H 5500 3900 50  0001 C CNN
 	1    5500 3900
