File: Hardware/HV9861A_SMPS/HV9861A_SMPS.sch (KiCad schematic (older format))
At the start: 22 parts

Commit message: Removed .bak. Refined schematic.
Parts:
- added C10, C11, C3, C4, C9: 47uF, symbol Device:CP1_Small
- added R1, R2: 0, symbol Device:R_Small
- added R3: 100, symbol Device:R_Small
- C6, C8: renamed from C?; symbol Device:C_Small -> Device:CP1_Small
- C7: renamed from C?; value 0.47uF -> 2.2uF
- D2: renamed from D?; value D -> 600V 2A
- R4: renamed from R?; value 0 -> 1k
- R5: renamed from R?; value 100k -> 50k
- gave numbers to parts that had none: 16
Connections:
- net GND: now also C3.2, C4.2
- net at C2.1, C6.1, C8.1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: now also C10.1, C11.1, C3.1, C4.1, C9.1
- net at C8.2, J3.2 (Pin_2), L1.1: now also C10.2, C11.2, C9.2
- net at U1.1: now also R3.2; no longer J2.1 (Pin_1)
- net at U1.2: now also R2.2; no longer J2.2 (Pin_2)
- new net: J2.1 (Pin_1), R1.1
- new net: J2.2 (Pin_2), R2.1
- new net: R1.2, R3.1
Other:
- moved on the sheet: J2, J3
